File: Hardware/Kicad/I2S.kicad_sch (KiCad schematic)
At the start: 10 parts, among them J2 MAX98357_AMPLIFIER_MODULE_OUT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, J31 MAX98357_AMPLIFIER_MODULE, J34 INMP441_LEFT, J35 INMP441_RIGHT, Q1 2N2222

Commit message: Inline accessors, small cleanups, removed empty destructors
Other:
- note added: "AUDIO"
- note removed: "I2S"
Changed lines of the file:
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@@
 		)
 	)
-	(text "I2S"
+	(text "AUDIO"
 		(exclude_from_sim no)
 		(at 104.902 26.67 0)

Commit message: Replaced 1602 to 2004 in Kicad and Tinkercad
Changed lines of the file:
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@@
+		)
+	)
+	(polyline
+		(pts
+			(xy 8.89 31.75) (xy 198.12 31.75)
+		)
+		(stroke
+			(width 0)
+			(type default)
 		)
 	)
@@
 		)
 	)
+	(polyline
+		(pts
+			(xy 10.16 160.02) (xy 199.39 160.02)
+		)
+		(stroke
+			(width 0)
+			(type default)
+		)
+	)
 	(wire
 		(pts
@@
 		)
 	)
+	(polyline
+		(pts
+			(xy 11.43 118.11) (xy 200.66 118.11)
+		)
+		(stroke
+			(width 0)
+			(type default)
+		)
+	)
 	(wire
 		(pts
@@
 		)
 		(stroke
+			(width 0)
+			(type default)
+		)
+	)
+	(polyline
+		(pts
+			(xy 10.16 80.01) (xy 199.39 80.01)
+		)
+		(stroke
