File: Hardware/Kicad/I2S.kicad_sch (KiCad schematic)
At the start: 10 parts, among them J2 MAX98357_AMPLIFIER_MODULE_OUT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, J31 MAX98357_AMPLIFIER_MODULE, J34 INMP441_LEFT, J35 INMP441_RIGHT, Q1 2N2222

Commit message: New Fraxis PCB layout
Parts:
- Q1: footprint PCM_Package_TO_SOT_THT_AKL:TO-92L_Inline_Wide_ECB -> Package_TO_SOT_SMD:TSOT-23_HandSoldering
Changed lines of the file:
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@@
 			)
 		)
-		(property "Footprint" "PCM_Package_TO_SOT_THT_AKL:TO-92L_Inline_Wide_ECB"
+		(property "Footprint" "Package_TO_SOT_SMD:TSOT-23_HandSoldering"
 			(at 114.3 135.89 0)
 			(hide yes)
