File: Hardware/Kicad/led_strips.kicad_sch (KiCad schematic)
At the start: 15 parts, among them J36 Led Strip 1 Begin, J37 Led Strip 2 Begin, J38 Led Strip 3 Begin, J39 Led Strip 4 Begin, J40 Led Strip 5 Begin, J42 Led Strip 1 End, J43 Led Strip 2 End, J44 Led Strip 3 End, J45 Led Strip 4 End, J46 Led Strip 5 End, U5 74AHCT125

Commit message: Replaced 1602 to 2004 in Kicad and Tinkercad
Changed lines of the file:
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@@
+		)
+	)
+	(polyline
+		(pts
+			(xy 11.43 68.58) (xy 200.66 68.58)
+		)
+		(stroke
+			(width 0)
+			(type default)
 		)
 	)
@@
 		)
 	)
+	(polyline
+		(pts
+			(xy 10.16 26.67) (xy 199.39 26.67)
+		)
+		(stroke
+			(width 0)
+			(type default)
+		)
+	)
 	(wire
 		(pts
@@
 		)
 		(stroke
+			(width 0)
+			(type default)
+		)
+	)
+	(polyline
+		(pts
+			(xy 11.43 100.33) (xy 200.66 100.33)
+		)
+		(stroke
+			(width 0)
+			(type default)
+		)
+	)
+	(polyline
+		(pts
+			(xy 10.16 138.43) (xy 199.39 138.43)
+		)
+		(stroke
