File: Hardware/Kicad/led_strips.kicad_sch (KiCad schematic)
At the start: 14 parts, among them J36 Led Strip 1 Begin, J37 Led Strip 2 Begin, J38 Led Strip 3 Begin, J39 Led Strip 4 Begin, J40 Led Strip 5 Begin, J42 Led Strip 1 End, J43 Led Strip 2 End, J44 Led Strip 3 End, J45 Led Strip 4 End, J46 Led Strip 5 End, U5 74AHCT125

Commit message: New Fraxis PCB layout
Other:
- note added: "1000 uf + 0.1 uF bij begin/eind"
Changed lines of the file:
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@@
+		)
+	)
+	(text "1000 uf + 0.1 uF bij begin/eind"
+		(exclude_from_sim no)
+		(at 159.766 164.592 0)
+		(effects
+			(font
+				(size 1.27 1.27)
+			)
 		)
 	)
