File: Hardware/Kicad/_autosave-1DGames.sch (KiCad schematic (older format))
At the start: 38 parts, among them J1 Conn_01x03, J2 Conn_01x02_Male, J3 Conn_01x04, J4 Conn_01x04, J5 Conn_01x04, J6 Conn_01x08, J7 Conn_01x08, J8 Conn_01x08, Q1 AO3401A, Q2 AO3401A, Q3 AO3401A, Q4 AO3401A, U1 ESP32-DEVKITC-32D, U2 74LS165, U3 74LS165

Commit message: New architecture, L1 composition finished, probably, on ESP32
Other:
- note added: "Main LCD Display 2004"
- note removed: "Main LCD Display 1602"
Changed lines of the file:
@@
 	8000 450  8000 11250
 Text Notes 5950 8050 0    79   Italic 16
-Main LCD Display 1602
+Main LCD Display 2004
 Text Notes 8400 750  0    79   Italic 16
 Switches and Pot Meters
