File: Hardware/Kicad/i2c.kicad_sch (KiCad schematic)
At the start: 25 parts, among them J17 MCP23017_Control, J22 MCP23017_Gpios, J32 LCD1602, U2 MCP23017x-x-SP, U3 BOB-12009

Commit message: Replaced 1602 to 2004 in Kicad and Tinkercad
Parts:
- C19: footprint (none) -> Capacitor_THT:CP_Radial_D5.0mm_P2.50mm
- J32: value LCD1602 -> LCD2004
- R26: value 4.7K -> 10K
Connections:
- net 3V3: now also C19.1
- net SYSTEM_BUTTON: no longer C19.1
Other:
- note added: "2004 I2C LCD DISPLAY MODULE"
- note removed: "1602 I2C LCD DISPLAY MODULE"
- moved on the sheet: C19, R20, R21, R22, R23, R24, R25, R26, R28

Commit message: New architecture, L1 composition finished, probably, on ESP32
Parts:
- added R29: 10K, Resistor_THT:R_Axial_DIN0204_L3.6mm_D1.6mm_P5.08mm_Horizontal, symbol Device:R
Connections:
- net 3V3: now also R29.2
- net MCP23017_INT_AB: now reaches U2.20 (INTA)
- net MCP23017_INT_AB: now also J22.3 (Pin_3), R29.1
- no-connect marks 10 -> 8
Other:
- note added: "Open Drain / Mirrored"
Changed lines of the file:
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@@
 	(generator_version "10.0")
 	(paper "A4" portrait)
+	(text "Open Drain / Mirrored\n"
+		(exclude_from_sim no)
+		(at 42.418 68.326 0)
+		(effects
+			(font
+				(size 1.27 1.27)
+			)
+		)
+	)
 	(text "For debouncing"
 		(exclude_from_sim no)
@@
 	(text "I2C LEVEL SHIFTER"
 		(exclude_from_sim no)
-		(at 109.474 167.894 0)
+		(at 109.22 166.116 0)
 		(effects
 			(font
@@
 	)
 	(junction
+		(at 39.37 60.96)
+		(diameter 0)
+		(color 0 0 0 0)
+	)
+	(junction
 		(at 170.18 83.82)
 		(diameter 0)
@@
 	)
 	(junction
-		(at 39.37 60.96)
+		(at 59.69 66.04)
 		(diameter 0)
 		(color 0 0 0 0)
@@
 	)
 	(no_connect
-		(at 125.73 130.81)
-	)
-	(no_connect
 		(at 91.44 181.61)
 	)
-	(no_connect
-		(at 59.69 66.04)
-	)
 	(wire
 		(pts
@@
 	(wire
 		(pts
+			(xy 59.69 63.5) (xy 59.69 66.04)
+		)
+		(stroke
+			(width 0)
+			(type default)
+		)
+	)
+	(wire
+		(pts
 			(xy 59.69 86.36) (xy 57.15 86.36)
 		)
@@
 	(wire
 		(pts
-			(xy 34.29 60.96) (xy 39.37 60.96)
+			(xy 35.56 60.96) (xy 39.37 60.96)
+		)
+		(stroke
+			(width 0)
+			(type default)
+		)
+	)
+	(wire
+		(pts
+			(xy 58.42 66.04) (xy 59.69 66.04)
 		)
 		(stroke
@@
 	(wire
 		(pts
-			(xy 125.73 128.27) (xy 148.59 128.27)
+			(xy 125.73 128.27) (xy 154.94 128.27)
 		)
 		(stroke
@@
 		)
 	)
+	(hierarchical_label "MCP23017_INT_AB"
+		(shape input)
+		(at 125.73 130.81 0)
+		(effects
+			(font
+				(size 1.27 1.27)
+			)
+			(justify left)
+		)
+	)
 	(hierarchical_label "I2C_SDA_3V3"
 		(shape input)
@@
 	(hierarchical_label "3V3"
 		(shape input)
-		(at 34.29 60.96 180)
+		(at 35.56 60.96 180)
+		(effects
+			(font
+				(size 1.27 1.27)
+			)
+			(justify right)
+		)
+	)
+	(hierarchical_label "3V3"
+		(shape input)
+		(at 52.07 63.5 180)
 		(effects
 			(font
@@
 		)
 	)
+	(hierarchical_label "MCP23017_INT_AB"
+		(shape input)
+		(at 58.42 66.04 180)
+		(effects
+			(font
+				(size 1.27 1.27)
+			)
+			(justify right)
+		)
+	)
 	(hierarchical_label "P2_JOYSTICK_DOWN"
 		(shape input)
@@
 	)
 	(symbol
+		(lib_id "Device:R")
+		(at 55.88 63.5 270)
+		(unit 1)
+		(body_style 1)
+		(exclude_from_sim no)
+		(in_bom yes)
+		(on_board yes)
+		(in_pos_files yes)
+		(dnp no)
+		(property "Reference" "R29"
+			(at 55.88 57.15 90)
+			(show_name no)
+			(do_not_autoplace no)
+			(effects
+				(font
+					(size 1.27 1.27)
+				)
+			)
+		)
+		(property "Value" "10K"
+			(at 55.88 59.944 90)
+			(show_name no)
+			(do_not_autoplace no)
+			(effects
+				(font
+					(size 1.27 1.27)
+				)
+			)
+		)
+		(property "Footprint" "Resistor_THT:R_Axial_DIN0204_L3.6mm_D1.6mm_P5.08mm_Horizontal"
+			(at 55.88 61.722 90)
+			(hide yes)
+			(show_name no)
+			(do_not_autoplace no)
+			(effects
+				(font
+					(size 1.27 1.27)
+				)
+			)
+		)
+		(property "Datasheet" ""
+			(at 55.88 63.5 0)
+			(hide yes)
+			(show_name no)
+			(do_not_autoplace no)
+			(effects
+				(font
+					(size 1.27 1.27)
+				)
+			)
+		)
+		(property "Description" "Resistor"
+			(at 55.88 63.5 0)
+			(hide yes)
+			(show_name no)
+			(do_not_autoplace no)
+			(effects
+				(font
+					(size 1.27 1.27)
+				)
+			)
+		)
+		(pin "2"
+		)
+		(pin "1"
+		)
+		(instances
+			(project "1DGames"
+				(path "/b1c649b1-f44d-46c7-9dea-818e75a1b87e/353760ae-7fc0-48a5-ab51-74b3f063c87e"
+					(reference "R29")
+					(unit 1)
+				)
+			)
+		)
+	)
+	(symbol
 		(lib_id "power:GND")
 		(at 127 194.31 0)
@@
 	(symbol
 		(lib_id "power:GND")
-		(at 148.59 128.27 0)
+		(at 154.94 128.27 0)
 		(unit 1)
 		(body_style 1)
@@
 		(fields_autoplaced yes)
 		(property "Reference" "#PWR021"
-			(at 148.59 134.62 0)
+			(at 154.94 134.62 0)
 			(hide yes)
 			(show_name no)
@@
 		)
 		(property "Value" "GND"
-			(at 148.59 133.35 0)
+			(at 154.94 133.35 0)
 			(show_name no)
 			(do_not_autoplace no)
@@
 		)
 		(property "Footprint" ""
-			(at 148.59 128.27 0)
+			(at 154.94 128.27 0)
 			(hide yes)
 			(show_name no)
@@
 		)
 		(property "Datasheet" ""
-			(at 148.59 128.27 0)
+			(at 154.94 128.27 0)
 			(hide yes)
 			(show_name no)
@@
 		)
 		(property "Description" "Power symbol creates a global label with name \"GND\" , ground"
-			(at 148.59 128.27 0)
+			(at 154.94 128.27 0)
 			(hide yes)
 			(show_name no)
