File: Hardware/Kicad/esp32.kicad_sch (KiCad schematic)
At the start: 9 parts, among them J5 Micro SD Card Reader, U1 AMS1117-3.3, U4 DEVKIT_V1_ESP32-WROOM-32, U6 ESP32-S3

Commit message: Replaced 1602 to 2004 in Kicad and Tinkercad
Connections:
- net CP_TM1637_DIN: now also U6.27 (GPIO21); no longer U6.18 (GPIO13/ADC2_CH2)
- net GND: now also U6.57 (GND)
- net I2C_SCL_3V3: now also U6.13 (GPIO8/ADC1_CH7); no longer U6.23 (GPIO17/ADC2_CH6)
- net I2C_SDA_3V3: now also U6.14 (GPIO9/ADC1_CH8)
- net I2S_BCLK: now also U6.15 (GPIO10/ADC1_CH9)
- net I2S_INMP441_DIN: now also U6.17 (GPIO12/ADC2_CH1)
- net I2S_MAX98357: now also U6.18 (GPIO13/ADC2_CH2); no longer U6.25 (GPIO19/USB_D-/ADC2_CH8)
- net I2S_WS_LRCLK: now also U6.16 (GPIO11/ADC2_CH0)
- net LED_STRIP_DATA_3V3: now also U6.36 (SPICLK_N/GPIO48); no longer U6.7 (GPIO2/ADC1_CH1)
- net P1_TM1637_DIN: now also U6.23 (GPIO17/ADC2_CH6); no longer U6.19 (GPIO14/ADC2_CH3)
- net P2_TM1637_DIN: now also U6.24 (GPIO18/ADC2_CH7); no longer U6.30 (SPIHD/GPIO27)
- net PASSIVE_BUZZER_SIGNAL: now also U6.19 (GPIO14/ADC2_CH3); no longer U6.9 (GPIO4/ADC1_CH3)
- net SPI_CS: now also U6.39 (GPIO34); no longer U6.38 (GPIO33)
- net SPI_MISO: now also U6.42 (GPIO37); no longer U6.35 (SPID/GPIO32)
- net SPI_MOSI: now also U6.40 (GPIO35)
- net SPI_SCK: now also U6.41 (GPIO36); no longer U6.28 (SPI_CS1/GPIO26)
- net TM1637_SHARED_CLK: now also U6.43 (GPIO38); no longer U6.24 (GPIO18/ADC2_CH7)
Other:
- moved on the sheet: U6
Changed lines of the file:
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@@
+		)
+	)
+	(polyline
+		(pts
+			(xy 10.16 152.4) (xy 199.39 152.4)
+		)
+		(stroke
+			(width 0)
+			(type default)
 		)
 	)
@@
 		)
 	)
+	(polyline
+		(pts
+			(xy 8.89 31.75) (xy 198.12 31.75)
+		)
+		(stroke
+			(width 0)
+			(type default)
+		)
+	)
 	(wire
 		(pts
@@
 		(pts
 			(xy 72.39 53.34) (xy 76.2 53.34)
+		)
+		(stroke
+			(width 0)
+			(type default)
+		)
+	)
+	(polyline
+		(pts
+			(xy 10.16 77.47) (xy 199.39 77.47)
 		)
 		(stroke
@@
 	)
 	(label "SPI_MISO"
-		(at 68.58 219.71 180)
+		(at 68.58 241.3 180)
 		(effects
 			(font
@@
 	)
 	(label "SPI_CS"
-		(at 68.58 222.25 180)
+		(at 68.58 233.68 180)
 		(effects
 			(font
@@
 	)
 	(label "SPI_MOSI"
-		(at 41.91 194.31 180)
+		(at 68.58 236.22 180)
 		(effects
 			(font
@@
 	)
 	(label "SPI_SCK"
-		(at 68.58 204.47 180)
+		(at 68.58 238.76 180)
 		(effects
 			(font
@@
 	(hierarchical_label "I2S_BCLK"
 		(shape output)
-		(at 165.1 213.36 0)
+		(at 134.62 210.82 0)
 		(effects
 			(font
@@
 	(hierarchical_label "I2S_WS_LRCLK"
 		(shape output)
-		(at 161.29 209.55 0)
+		(at 134.62 213.36 0)
 		(effects
 			(font
@@
 	(hierarchical_label "CP_TM1637_DIN"
 		(shape output)
-		(at 134.62 209.55 0)
+		(at 134.62 228.6 0)
 		(effects
 			(font
@@
 	(hierarchical_label "I2S_MAX98357"
 		(shape output)
-		(at 134.62 171.45 0)
+		(at 134.62 218.44 0)
 		(effects
 			(font
@@
 	(hierarchical_label "TM1637_SHARED_CLK"
 		(shape output)
-		(at 134.62 217.17 0)
+		(at 134.62 231.14 0)
 		(effects
 			(font
@@
 	(hierarchical_label "I2C_SCL_3V3"
 		(shape output)
-		(at 134.62 214.63 0)
+		(at 134.62 205.74 0)
 		(effects
 			(font
@@
 	(hierarchical_label "P2_TM1637_DIN"
 		(shape output)
-		(at 68.58 207.01 180)
-		(effects
-			(font
-				(size 1.27 1.27)
-			)
-			(justify right)
+		(at 134.62 226.06 0)
+		(effects
+			(font
+				(size 1.27 1.27)
+			)
+			(justify left)
 		)
 	)
@@
 	(hierarchical_label "P1_TM1637_DIN"
 		(shape output)
-		(at 134.62 212.09 0)
+		(at 134.62 223.52 0)
 		(effects
 			(font
@@
 	(hierarchical_label "I2C_SDA_3V3"
 		(shape bidirectional)
-		(at 156.21 203.2 0)
+		(at 134.62 208.28 0)
 		(effects
 			(font
@@
 	(hierarchical_label "LED_STRIP_DATA_3V3"
 		(shape output)
-		(at 134.62 181.61 0)
+		(at 134.62 241.3 0)
 		(effects
 			(font
@@
 	(hierarchical_label "5V_BOARD"
 		(shape input)
-		(at 104.14 156.21 90)
+		(at 104.14 165.1 90)
 		(effects
 			(font
@@
 	(hierarchical_label "I2S_INMP441_DIN"
 		(shape input)
-		(at 157.48 205.74 0)
+		(at 134.62 215.9 0)
 		(effects
 			(font
@@
 	(hierarchical_label "PASSIVE_BUZZER_SIGNAL"
 		(shape output)
-		(at 134.62 186.69 0)
+		(at 134.62 220.98 0)
 		(effects
 			(font
@@
 	)
 	(symbol
+		(lib_name "GND_3")
+		(lib_id "power:GND")
+		(at 101.6 246.38 0)
+		(mirror y)
+		(unit 1)
+		(body_style 1)
+		(exclude_from_sim no)
+		(in_bom yes)
+		(on_board yes)
+		(in_pos_files yes)
+		(dnp no)
+		(property "Reference" "#PWR048"
+			(at 101.6 252.73 0)
+			(hide yes)
+			(show_name no)
+			(do_not_autoplace no)
+			(effects
+				(font
+					(size 1.27 1.27)
+				)
+			)
+		)
+		(property "Value" "GND"
+			(at 101.473 250.7742 0)
+			(show_name no)
+			(do_not_autoplace no)
+			(effects
+				(font
+					(size 1.27 1.27)
+				)
+			)
+		)
+		(property "Footprint" ""
+			(at 101.6 246.38 0)
+			(hide yes)
+			(show_name no)
+			(do_not_autoplace no)
+			(effects
+				(font
+					(size 1.27 1.27)
+				)
+			)
+		)
+		(property "Datasheet" ""
+			(at 101.6 246.38 0)
+			(hide yes)
+			(show_name no)
+			(do_not_autoplace no)
+			(effects
+				(font
+					(size 1.27 1.27)
+				)
+			)
+		)
+		(property "Description" ""
+			(at 101.6 246.38 0)
+			(show_name no)
+			(do_not_autoplace no)
+			(effects
+				(font
+					(size 1.27 1.27)
+				)
+			)
+		)
+		(pin "1"
+		)
+		(instances
+			(project "1DGames"
+				(path "/b1c649b1-f44d-46c7-9dea-818e75a1b87e/baa69087-af62-4829-89ca-50abd72c3450"
+					(reference "#PWR048")
+					(unit 1)
+				)
+			)
+		)
+	)
+	(symbol
 		(lib_name "GND_2")
 		(lib_id "power:GND")
@@
 	(symbol
 		(lib_id "PCM_Espressif:ESP32-S3")
-		(at 101.6 196.85 0)
+		(at 101.6 205.74 0)
 		(unit 1)
 		(body_style 1)
@@
 		(fields_autoplaced yes)
 		(property "Reference" "U6"
-			(at 103.7433 237.49 0)
+			(at 103.7433 246.38 0)
 			(show_name no)
 			(do_not_autoplace no)
@@
 		)
 		(property "Value" "ESP32-S3"
-			(at 103.7433 240.03 0)
+			(at 103.7433 248.92 0)
 			(show_name no)
 			(do_not_autoplace no)
@@
 		)
 		(property "Footprint" "Package_DFN_QFN:QFN-56-1EP_7x7mm_P0.4mm_EP5.6x5.6mm"
-			(at 101.6 245.11 0)
+			(at 101.6 254 0)
 			(hide yes)
 			(show_name no)
@@
 		)
 		(property "Datasheet" "https://www.espressif.com/sites/default/files/documentation/esp32-s3_datasheet_en.pdf"
-			(at 101.6 247.65 0)
+			(at 101.6 256.54 0)
 			(hide yes)
 			(show_name no)
@@
 		)
 		(property "Description" "ESP32-S3 is a low-power MCU-based system-on-chip (SoC) that supports 2.4 GHz Wi-Fi and Bluetooth® Low Energy (Bluetooth LE). It consists of high-performance dual-core microprocessor (Xtensa® 32-bit LX7), a low power coprocessor, a Wi-Fi baseband, a Bluetooth LE baseband, RF module, and peripherals."
-			(at 101.6 196.85 0)
+			(at 101.6 205.74 0)
 			(hide yes)
 			(show_name no)
@@
 					(unit 1)
 				)
-			)
-		)
-	)
-	(symbol
-		(lib_name "GND_3")
-		(lib_id "power:GND")
-		(at 154.94 156.21 0)
-		(mirror y)
-		(unit 1)
-		(body_style 1)
-		(exclude_from_sim no)
-		(in_bom yes)
-		(on_board yes)
-		(in_pos_files yes)
-		(dnp no)
-		(property "Reference" "#PWR046"
-			(at 154.94 162.56 0)
-			(hide yes)
-			(show_name no)
-			(do_not_autoplace no)
-			(effects
-				(font
-					(size 1.27 1.27)
-				)
-			)
-		)
-		(property "Value" "GND"
-			(at 154.813 160.6042 0)
-			(show_name no)
-			(do_not_autoplace no)
-			(effects
-				(font
-					(size 1.27 1.27)
-				)
-			)
-		)
-		(property "Footprint" ""
-			(at 154.94 156.21 0)
-			(hide yes)
-			(show_name no)
-			(do_not_autoplace no)
-			(effects
-				(font
-					(size 1.27 1.27)
-				)
-			)
-		)
-		(property "Datasheet" ""
-			(at 154.94 156.21 0)
-			(hide yes)
-			(show_name no)
-			(do_not_autoplace no)
-			(effects
-				(font
-					(size 1.27 1.27)
-				)
-			)
-		)
-		(property "Description" ""
-			(at 154.94 156.21 0)
-			(show_name no)
-			(do_not_autoplace no)
-			(effects
-				(font
-					(size 1.27 1.27)
-				)
-			)
-		)
-		(pin "1"
-		)
-		(instances
-			(project "1DGames"
-				(path "/b1c649b1-f44d-46c7-9dea-818e75a1b87e/baa69087-af62-4829-89ca-50abd72c3450"
-					(reference "#PWR046")
-					(unit 1)
-				)

Commit message: New architecture, L1 composition finished, probably, on ESP32
Connections:
- net MCP23017_INT_AB: now reaches U4.13 (IO12)
- net MCP23017_INT_AB: now also U6.6 (GPIO1/ADC1_CH0)
- no-connect marks 18 -> 53
Changed lines of the file:
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@@
+	)
+	(no_connect
+		(at 68.58 218.44)
 	)
 	(no_connect
@@
 	)
 	(no_connect
+		(at 68.58 182.88)
+	)
+	(no_connect
+		(at 68.58 208.28)
+	)
+	(no_connect
+		(at 134.62 195.58)
+	)
+	(no_connect
 		(at 119.38 119.38)
 	)
 	(no_connect
+		(at 68.58 226.06)
+	)
+	(no_connect
+		(at 68.58 177.8)
+	)
+	(no_connect
+		(at 68.58 190.5)
+	)
+	(no_connect
+		(at 68.58 205.74)
+	)
+	(no_connect
+		(at 96.52 165.1)
+	)
+	(no_connect
+		(at 134.62 238.76)
+	)
+	(no_connect
 		(at 119.38 134.62)
 	)
 	(no_connect
+		(at 134.62 190.5)
+	)
+	(no_connect
+		(at 68.58 228.6)
+	)
+	(no_connect
+		(at 99.06 165.1)
+	)
+	(no_connect
 		(at 78.74 134.62)
 	)
@@
 	)
 	(no_connect
+		(at 134.62 180.34)
+	)
+	(no_connect
+		(at 134.62 172.72)
+	)
+	(no_connect
+		(at 101.6 165.1)
+	)
+	(no_connect
 		(at 78.74 109.22)
 	)
 	(no_connect
+		(at 68.58 203.2)
+	)
+	(no_connect
+		(at 134.62 200.66)
+	)
+	(no_connect
+		(at 134.62 193.04)
+	)
+	(no_connect
 		(at 119.38 139.7)
 	)
@@
 	)
 	(no_connect
+		(at 134.62 170.18)
+	)
+	(no_connect
 		(at 78.74 101.6)
 	)
 	(no_connect
-		(at 78.74 127)
+		(at 134.62 177.8)
+	)
+	(no_connect
+		(at 134.62 233.68)
+	)
+	(no_connect
+		(at 134.62 198.12)
+	)
+	(no_connect
+		(at 68.58 200.66)
 	)
 	(no_connect
@@
 	)
 	(no_connect
+		(at 68.58 193.04)
+	)
+	(no_connect
+		(at 134.62 185.42)
+	)
+	(no_connect
+		(at 134.62 203.2)
+	)
+	(no_connect
 		(at 78.74 96.52)
 	)
@@
 	)
 	(no_connect
+		(at 68.58 185.42)
+	)
+	(no_connect
+		(at 68.58 231.14)
+	)
+	(no_connect
+		(at 93.98 165.1)
+	)
+	(no_connect
 		(at 119.38 137.16)
 	)
@@
 	)
 	(no_connect
+		(at 68.58 213.36)
+	)
+	(no_connect
+		(at 134.62 236.22)
+	)
+	(no_connect
+		(at 68.58 215.9)
+	)
+	(no_connect
+		(at 68.58 170.18)
+	)
+	(no_connect
 		(at 78.74 99.06)
 	)
 	(no_connect
+		(at 68.58 220.98)
+	)
+	(no_connect
 		(at 78.74 139.7)
+	)
+	(no_connect
+		(at 68.58 223.52)
 	)
 	(wire
@@
 		(shape output)
 		(at 134.62 213.36 0)
+		(effects
+			(font
+				(size 1.27 1.27)
+			)
+			(justify left)
+		)
+	)
+	(hierarchical_label "MCP23017_INT_AB"
+		(shape input)
+		(at 134.62 187.96 0)
 		(effects
 			(font
@@
 		)
 	)
+	(hierarchical_label "MCP23017_INT_AB"
+		(shape input)
+		(at 78.74 127 180)
+		(effects
+			(font
+				(size 1.27 1.27)
+			)
+			(justify right)
+		)
+	)

Commit message: Broken code, halfway joystick gdi
Connections:
- net HC_SR04_TRIG_2: now reaches U6.10 (GPIO5/ADC1_CH4)
- net HC_SR04_TRIG_3: now reaches U6.28 (SPI_CS1/GPIO26)
- net HC_SR04_ECHO_3: now reaches U6.30 (SPIHD/GPIO27)
- net HC_SR04_ECHO_2: now reaches U6.35 (SPID/GPIO32)
- net HC_SR04_ECHO_1: now reaches U6.38 (GPIO33)
- net HC_SR04_ECHO_4: now reaches U6.51 (GPIO45)
- net HC_SR04_TRIG_4: now reaches U6.7 (GPIO2/ADC1_CH1)
- net HC_SR04_TRIG_1: now reaches U6.9 (GPIO4/ADC1_CH3)
- no-connect marks 53 -> 45
Changed lines of the file:
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@@
-	)
-	(no_connect
-		(at 134.62 195.58)
 	)
 	(no_connect
@@
 	)
 	(no_connect
-		(at 134.62 190.5)
-	)
-	(no_connect
-		(at 68.58 228.6)
-	)
-	(no_connect
 		(at 99.06 165.1)
 	)
@@
 	)
 	(no_connect
-		(at 134.62 233.68)
-	)
-	(no_connect
-		(at 134.62 198.12)
-	)
-	(no_connect
 		(at 68.58 200.66)
 	)
@@
 	)
 	(no_connect
-		(at 68.58 231.14)
-	)
-	(no_connect
 		(at 93.98 165.1)
 	)
@@
 	)
 	(no_connect
-		(at 68.58 213.36)
-	)
-	(no_connect
 		(at 134.62 236.22)
-	)
-	(no_connect
-		(at 68.58 215.9)
 	)
 	(no_connect
@@
 		(shape output)
 		(at 134.62 210.82 0)
+		(effects
+			(font
+				(size 1.27 1.27)
+			)
+			(justify left)
+		)
+	)
+	(hierarchical_label "HC_SR04_ECHO_1"
+		(shape input)
+		(at 68.58 231.14 180)
+		(effects
+			(font
+				(size 1.27 1.27)
+			)
+			(justify right)
+		)
+	)
+	(hierarchical_label "HC_SR04_TRIG_4"
+		(shape output)
+		(at 134.62 190.5 0)
 		(effects
 			(font
@@
 		)
 	)
+	(hierarchical_label "HC_SR04_TRIG_3"
+		(shape output)
+		(at 68.58 213.36 180)
+		(effects
+			(font
+				(size 1.27 1.27)
+			)
+			(justify right)
+		)
+	)
 	(hierarchical_label "5V_BOARD"
 		(shape input)
@@
 		)
 	)
+	(hierarchical_label "HC_SR04_ECHO_3"
+		(shape input)
+		(at 68.58 215.9 180)
+		(effects
+			(font
+				(size 1.27 1.27)
+			)
+			(justify right)
+		)
+	)
 	(hierarchical_label "I2C_SCL_3V3"
 		(shape output)
@@
 		)
 	)
+	(hierarchical_label "HC_SR04_TRIG_1"
+		(shape output)
+		(at 134.62 195.58 0)
+		(effects
+			(font
+				(size 1.27 1.27)
+			)
+			(justify left)
+		)
+	)
 	(hierarchical_label "P1_TM1637_DIN"
 		(shape output)
@@
 			)
 			(justify left)
+		)
+	)
+	(hierarchical_label "HC_SR04_ECHO_2"
+		(shape input)
+		(at 68.58 228.6 180)
+		(effects
+			(font
+				(size 1.27 1.27)
+			)
+			(justify right)
 		)
 	)
@@
 		(effects
 			(font
+				(size 1.27 1.27)
+			)
+			(justify left)
+		)
+	)
+	(hierarchical_label "HC_SR04_ECHO_4"
+		(shape input)
+		(at 134.62 233.68 0)
+		(effects
+			(font
+				(size 1.27 1.27)
+			)
+			(justify left)
+		)
+	)
+	(hierarchical_label "HC_SR04_TRIG_2"
+		(shape output)
+		(at 134.62 198.12 0)
+		(effects
+			(font
