File: Hardware/Kicad/power.kicad_pcb (KiCad board)
At the start: 2 copper layers, 80.3 x 60.1 mm, 22 parts, among them J1 PinHeader_01x05_P2.54mm_Verti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, J10 LED Strips Output, J12 Enclosure Power, J13 PCB Power, J2 PinHeader_01x05_P2.54mm_Verti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, J9 Power In, U1 AMS1117-3.3

Commit message: Added safety in Kicad power, added NVS read version/tm1637 brightness
Parts:
- added D2: SMAJ5.0A, PCM_Diode_SMD_AKL:D_SMA, F.Cu at (159.4, 50.0)
Routing:
- net Net-(D1-A): track 96.8 -> 107.8 mm
- net GND: track 234.9 -> 239.6 mm, vias 1 -> 2
Other:
- board text added: "80x60mm"
