File: Hardware/Kicad_Board/i2c.kicad_sch (KiCad schematic)
At the start: 23 parts, among them J17 MCP23017_Control, J22 MCP23017_Gpios, J32 LCD2004, U2 MCP23017x-x-SP, U3 BOB-12009

Commit message: Added Kicad proto board
Parts:
- added R1, R2: 4.7K, Resistor_THT:R_Axial_DIN0204_L3.6mm_D1.6mm_P5.08mm_Horizontal, symbol Device:R
- added R29: 10K, Resistor_THT:R_Axial_DIN0204_L3.6mm_D1.6mm_P5.08mm_Horizontal, symbol Device:R
- C19: value 0.1uF -> 100nF; footprint Capacitor_SMD:C_0805_2012Metric_Pad1.18x1.45mm_HandSolder -> Capacitor_THT:CP_Radial_D5.0mm_P2.50mm
- R17, R18, R19, R20, R21, R22, R23, R24, R25, R26, R28: footprint PCM_Resistor_SMD_AKL:R_0805_2012Metric_Pad1.20x1.40mm_HandSolder -> Resistor_THT:R_Axial_DIN0204_L3.6mm_D1.6mm_P5.08mm_Horizontal
- R3, R4, R5, R6, R7: value 270 -> 220-270; footprint PCM_Resistor_SMD_AKL:R_0805_2012Metric_Pad1.20x1.40mm_HandSolder -> Resistor_THT:R_Axial_DIN0204_L3.6mm_D1.6mm_P5.08mm_Horizontal
Connections:
- net 3V3: now also R1.1, R2.2, R29.2
- net I2C_SCL_3V3: now also R1.2
- net I2C_SDA_3V3: now also R2.1
- net MCP23017_INT_AB: now also R29.1
- net 5V_RAIL: now reaches C13.2, J32.1 (Pin_1)
- net 5V renamed 5V_BOARD
