File: Hardware/Kicad_Board/led_strips.kicad_sch (KiCad schematic)
At the start: 14 parts, among them J36 Led Strip 1 Begin, J37 Led Strip 2 Begin, J38 Led Strip 3 Begin, J39 Led Strip 4 Begin, J40 Led Strip 5 Begin, J42 Led Strip 1 End, J43 Led Strip 2 End, J44 Led Strip 3 End, J45 Led Strip 4 End, J46 Led Strip 5 End, U5 74AHCT125

Commit message: Added Kicad proto board
Parts:
- added C15: 1000 uF, Capacitor_THT:CP_Radial_D10.0mm_P2.50mm, symbol Device:C
- C16, C17: footprint Capacitor_SMD:C_0805_2012Metric_Pad1.18x1.45mm_HandSolder -> Capacitor_THT:C_Disc_D3.0mm_W1.6mm_P2.50mm
- J36: footprint Connector_AMASS:AMASS_MR30PW-FB_1x03_P3.50mm_Horizontal -> PCM_SparkFun-Connector:ScrewTerminal_1x03_P5.0mm; now in the parts list
- J42: footprint (none) -> PCM_SparkFun-Connector:ScrewTerminal_1x03_P5.0mm
- R8: footprint PCM_Resistor_SMD_AKL:R_0805_2012Metric_Pad1.20x1.40mm_HandSolder -> Resistor_THT:R_Axial_DIN0204_L3.6mm_D1.6mm_P5.08mm_Horizontal
Connections:
- net 5V: now also J36.1 (Pin_1), J37.1 (Pin_1), J38.1 (Pin_1), J39.1 (Pin_1), J40.1 (Pin_1), J42.1 (Pin_1), J43.1 (Pin_1), J44.1 (Pin_1), J45.1 (Pin_1), J46.1 (Pin_1), C15.1; no longer C16.1, C17.1, J36.3 (Pin_3), J37.3 (Pin_3), J38.3 (Pin_3), J39.3 (Pin_3), J40.3 (Pin_3), J42.3 (Pin_3), J43.3 (Pin_3), J44.3 (Pin_3), J45.3 (Pin_3), J46.3 (Pin_3), U5.10, U5.13, U5.14 (VCC), U5.4
- net GND: now also C15.2
- net LED_STRIP_DATA_1_TO_2_5V: now also J37.3 (Pin_3), J42.3 (Pin_3); no longer J37.1 (Pin_1), J42.1 (Pin_1)
- net LED_STRIP_DATA_2_TO_3_5V: now also J38.3 (Pin_3), J43.3 (Pin_3); no longer J38.1 (Pin_1), J43.1 (Pin_1)
- net LED_STRIP_DATA_3_TO_4_5V: now also J39.3 (Pin_3), J44.3 (Pin_3); no longer J39.1 (Pin_1), J44.1 (Pin_1)
- net LED_STRIP_DATA_4_to_5_5V: now also J40.3 (Pin_3), J45.3 (Pin_3); no longer J40.1 (Pin_1), J45.1 (Pin_1)
- net LED_STRIP_DATA_5V: now also J36.3 (Pin_3); no longer J36.1 (Pin_1)
- new net 5V_BOARD: C16.1, C17.1, U5.10, U5.13, U5.14 (VCC), U5.4
Other:
- note added: "Cap is not attached on a proto board"
